File: STM32G431 Dev Board.kicad_pcb (KiCad board)
At the start: 2 copper layers, 30 x 64.6 mm, 40 parts, among them J1 Conn_02x04_Counter_Clockwise, J2 USB_C_Receptacle_USB2.0_16P, J3 Conn_02x11_Odd_Even, J4 Conn_02x11_Odd_Even, SW1 RST, SW2 BOOT, SW3 USER, U1 STM32G431CBTx, U2 USBLC6-2SC6, Y1 Crystal_GND24

Commit message: changed pin order
Parts:
- J3, J4: value Conn_02x11_Odd_Even -> Conn_01x22; footprint Connector_PinHeader_2.54mm:PinHeader_2x11_P2.54mm_Vertical -> Connector_PinHeader_2.54mm:PinHeader_1x22_P2.54mm_Vertical
- moved D3 43.8 mm to (158.6, 105.6), turned to 90 degrees
- moved J3 42.0 mm to (170.3, 56.7), turned to 0 degrees
- moved J4 40.4 mm to (198.2, 56.7), turned to 0 degrees
- moved R4 40.2 mm to (158.7, 102.2), turned to -90 degrees
- moved C12 23.3 mm to (186.3, 68.2)
- moved Y1 22.8 mm to (185.6, 70.6)
- moved R2 22.7 mm to (180.7, 68.9), turned to 90 degrees
- moved C13 22.6 mm to (182.9, 71.0)
- moved J1 18.5 mm to (194.6, 101.8)
- moved D2 18.0 mm to (180.7, 65.6), turned to -90 degrees
- moved JP1 17.9 mm to (187.1, 74.4), turned to -90 degrees
- moved JP2 16.9 mm to (184.2, 74.4), turned to -90 degrees
- moved C15 15.7 mm to (190.7, 76.4), turned to 0 degrees
- moved C4 14.3 mm to (190.7, 78.4), turned to 0 degrees
- moved JP4 13.5 mm to (175.8, 74.8)
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Connections:
- J3 pad 10: /PA5 -> /PC14
- J3 pad 11: /PA6 -> /PC15
- J3 pad 12: /PA7 -> /PA0
- J3 pad 13: /PA8 -> /PA1
- J3 pad 14: /PA9 -> /PA4
- J3 pad 15: /PA10 -> /PA5
- J3 pad 16: /PA15 -> /PA6
- J3 pad 17: /PF0_GPIO -> /PA7
- J3 pad 18: /PF1_GPIO -> /PA8
- J3 pad 19: /PC13 -> /PA9
- J3 pad 2: GND -> /VDD
- J3 pad 20: /PC14 -> /PA10
- J3 pad 21: /PC15 -> /PA15
- J3 pad 5: /VDD -> GND
- J3 pad 7: /PA0 -> /PF0_GPIO
- J3 pad 8: /PA1 -> /PF1_GPIO
- J3 pad 9: /PA4 -> /PC13
- J4 pad 2: GND -> /VBUS
- J4 pad 3: /VBUS -> GND
Routing:
- net /VDD: track 96.5 -> 36.6 mm, vias 6 -> 0
- net /NRST: track 18.5 -> 53.6 mm
- net /PC13: track 8.94 -> 33.1 mm, vias 0 -> 2
- net /PA15: track 23.1 -> 43.6 mm, vias 2 -> 4
- net /BOOT0: track 27.6 -> 47.6 mm, vias 2 -> 4
- net /PB6: track 27.3 -> 9.60 mm, vias 2 -> 1
- net /PA7: track 8.20 -> 23.0 mm, vias 2 -> 0
- net /PA6: track 6.42 -> 21.1 mm, vias 2 -> 0
- net /PA4: track 8.16 -> 22.7 mm
- net /PB7: track 24.1 -> 10.1 mm
- net /PA11: track 7.12 -> 20.8 mm
- net /PB4: track 27.1 -> 13.5 mm, vias 2 -> 1
- net /PB5: track 24.5 -> 11.6 mm, vias 2 -> 1
- net /PA12: track 7.21 -> 20.1 mm
- net /PB15: track 15.5 -> 28.3 mm, vias 0 -> 2
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- added copper zone on B.Cu, net GND
Other:
- board size 30 x 64.6 mm -> 31.3 x 60 mm

Commit message: most routing done
Parts:
- moved D3 45.3 mm to (190.5, 73.5)
- moved R4 44.3 mm to (192.4, 73.5), turned to 90 degrees
- moved J2 12.6 mm to (190.2, 111.0)
- moved R5 12.6 mm to (188.9, 104.0)
- moved R6 12.6 mm to (192.2, 104.0)
- moved U2 12.6 mm to (190.2, 102.1)
- moved J1 12.4 mm to (182.2, 102.0)
- moved R2 11.7 mm to (192.4, 69.7)
- moved D2 10.6 mm to (190.5, 69.7), turned to 90 degrees
- moved C11 9.45 mm to (190.2, 96.7), turned to 180 degrees
- moved C10 8.11 mm to (190.4, 98.7), turned to 180 degrees
- moved C9 4.59 mm to (183.1, 97.1), turned to 90 degrees
- moved PS1 3.51 mm to (186.3, 97.8)
- moved C8 2.64 mm to (181.3, 97.1), turned to 90 degrees
- moved JP4 1.35 mm to (176.9, 75.6)
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Connections:
- J3 pad 1: /VDD -> GND
- J3 pad 10: /PC14 -> /PA5
- J3 pad 11: /PC15 -> /PA6
- J3 pad 12: /PA0 -> /PA7
- J3 pad 13: /PA1 -> /PA8
- J3 pad 14: /PA4 -> /PA9
- J3 pad 15: /PA5 -> /PA10
- J3 pad 16: /PA6 -> /PA15
- J3 pad 17: /PA7 -> GND
- J3 pad 18: /PA8 -> GND
- J3 pad 19: /PA9 -> GND
- J3 pad 2: /VDD -> /PF0_GPIO
- J3 pad 20: /PA10 -> /VDD
- J3 pad 21: /PA15 -> /VDD
- J3 pad 22: GND -> /VDD
- J3 pad 3: /VDD -> /PF1_GPIO
- J3 pad 4: GND -> /PC13
- J3 pad 5: GND -> /PC14
- J3 pad 6: GND -> /PC15
- J3 pad 7: /PF0_GPIO -> /PA0
- J3 pad 8: /PF1_GPIO -> /PA1
- J3 pad 9: /PC13 -> /PA4
- J4 pad 1: /VBUS -> /VDD
- J4 pad 10: /PB5 -> /PB7
- J4 pad 11: /PB6 -> /BOOT0
- J4 pad 12: /PB7 -> /PB9
- J4 pad 13: /BOOT0 -> /PB10
- J4 pad 14: /PB9 -> /PB11
- J4 pad 15: /PB10 -> /PB12
- J4 pad 16: /PB11 -> /PB13
- J4 pad 17: /PB12 -> /PB14
- J4 pad 18: /PB13 -> /PB15
- J4 pad 19: /PB14 -> GND
- J4 pad 2: /VBUS -> GND
- J4 pad 20: /PB15 -> GND
- J4 pad 21: /VDD -> /VBUS
- J4 pad 22: GND -> /VBUS
- J4 pad 3: GND -> /PB0
- J4 pad 4: GND -> /PB1
- J4 pad 5: /PB0 -> /PB2
- J4 pad 6: /PB1 -> /PB3
- J4 pad 7: /PB2 -> /PB4
- J4 pad 8: /PB3 -> /PB5
- J4 pad 9: /PB4 -> /PB6
Routing:
- net /VDD: track 36.6 -> 153.0 mm, vias 0 -> 10
- net /PB2: track 15.5 -> 33.6 mm, vias 2 -> 6
- net /PA15: track 43.6 -> 32.2 mm, vias 4 -> 2
- net /PF1_GPIO: track 4.99 -> 16.3 mm
- net /PF0_GPIO: track 4.91 -> 16.0 mm
- net /PC13: track 33.1 -> 43.3 mm
- net /PA7: track 23.0 -> 12.9 mm
- net /PA6: track 21.1 -> 11.4 mm
- net /PA14: track 24.4 -> 33.4 mm, vias 2 -> 0
- net /PA13: track 20.5 -> 29.4 mm, vias 2 -> 0
- net /PA5: track 19.1 -> 11.2 mm
- net /PA4: track 22.7 -> 14.8 mm
- net /PA10: track 27.6 -> 20.6 mm
- net /PC14: track 19.8 -> 26.3 mm
- net Net-(PS1-EN): track 11.9 -> 6.50 mm
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- added copper zone on F.Cu, net GND
