File: STM32G431 Dev Board.kicad_sch (KiCad schematic)
At the start: 0 parts

Commit message: first layout
Parts:
- added C1, C10, C14, C15, C4, C5, C6, C7, C9: 100n, Capacitor_SMD:C_0603_1608Metric, symbol Device:C
- added C11: 10u, Capacitor_SMD:C_0805_2012Metric, symbol Device:C
- added C12, C13: 6.8p, Capacitor_SMD:C_0402_1005Metric, symbol Device:C
- added C2, C8: 1u, Capacitor_SMD:C_0603_1608Metric, symbol Device:C
- added C3: 4.7u, Capacitor_SMD:C_0805_2012Metric, symbol Device:C
- added D1: D_TVS, Diode_SMD:D_SOD-323, symbol Device:D_TVS
- added D2: blue, LED_SMD:LED_0603_1608Metric, symbol Device:LED
- added D3: red, LED_SMD:LED_0603_1608Metric, symbol Device:LED
- added J1: Conn_02x04_Counter_Clockwise, Connector_PinHeader_2.54mm:PinHeader_2x04_P2.54mm_Horizontal, symbol Connector_Generic:Conn_02x04_Counter_Clockwise
- added J2: USB_C_Receptacle_USB2.0_16P, Connector_USB:USB_C_Receptacle_HRO_TYPE-C-31-M-12, symbol Connector:USB_C_Receptacle_USB2.0_16P
- added J3, J4: Conn_02x11_Odd_Even, Connector_PinHeader_2.54mm:PinHeader_2x11_P2.54mm_Vertical, symbol Connector_Generic:Conn_02x11_Odd_Even
- added JP1, JP2: SolderJumper_2_Open, Jumper:SolderJumper-2_P1.3mm_Open_Pad1.0x1.5mm, symbol Jumper:SolderJumper_2_Open
- added JP3, JP4: SolderJumper_2_Bridged, Jumper:SolderJumper-2_P1.3mm_Bridged2Bar_Pad1.0x1.5mm, symbol Jumper:SolderJumper_2_Bridged
- added L1: 600R@100MHz, Inductor_SMD:L_0603_1608Metric, symbol Device:L
- added PS1: LD39050PU33R, SON95P300X300X100-7N-D, symbol LD39050PU33R:LD39050PU33R
- added R1: 10k, Resistor_SMD:R_0603_1608Metric, symbol Device:R
- added R2, R4: 2.2k, Resistor_SMD:R_0603_1608Metric, symbol Device:R
- added R3: 1k, Resistor_SMD:R_0603_1608Metric, symbol Device:R
- added R5, R6: 5.1k, Resistor_SMD:R_0603_1608Metric, symbol Device:R
- added SW1: RST, Button_Switch_SMD:SW_SPST_TL3342, symbol Switch:SW_Push
- added SW2: BOOT, Button_Switch_SMD:SW_SPST_TL3342, symbol Switch:SW_Push
- added SW3: USER, Button_Switch_SMD:SW_SPST_TL3342, symbol Switch:SW_Push
- added U1: STM32G431CBTx, Package_QFP:LQFP-48_7x7mm_P0.5mm, symbol MCU_ST_STM32G4:STM32G431CBTx
- added U2: USBLC6-2SC6, Package_TO_SOT_SMD:SOT-23-6, symbol Power_Protection:USBLC6-2SC6
- added Y1: Crystal_GND24, Crystal:Crystal_SMD_3225-4Pin_3.2x2.5mm, symbol Device:Crystal_GND24
Connections:
- new net: R3.1, SW3.2
- new net: D3.2 (A), R4.2
- new net: C12.2, JP1.1 (A), Y1.3
- new net: C10.2, C11.2, PS1.1 (EN), PS1.6 (VIN)
- new net: C13.2, JP2.1 (A), Y1.1
- new net: D2.2 (A), R2.2
- new net: J2.A5 (CC1), R5.2
- new net: J2.B5 (CC2), R6.2
- new net BOOT0: J4.13 (Pin_13), R1.2, SW2.2, U1.45 (PB8)
- new net D+: J2.A6 (D+), J2.B6 (D+), U2.3 (I/O2)
- new net D-: J2.A7 (D-), J2.B7 (D-), U2.1 (I/O1)
- new net GND: C1.2, C12.1, C13.1, C14.2, C15.2, C2.2, C3.2, C4.2, C5.2, C6.2, C7.2, C8.2, C9.2, D1.2 (A2), D2.1 (K), D3.1 (K), J1.2 (Pin_2), J1.7 (Pin_7), J2.A1 (GND), J2.A12 (GND), J2.B1 (GND), J2.B12 (GND), J2.SH (SHIELD), J3.2 (Pin_2), J3.22 (Pin_22), J3.4 (Pin_4), J3.6 (Pin_6), J4.2 (Pin_2), J4.22 (Pin_22), J4.4 (Pin_4), PS1.2 (GND), PS1.7 (PAD), R1.1, R5.1, R6.1, SW1.2, U1.19 (VSSA), U1.23 (VSS), U1.35 (VSS), U1.47 (VSS), U2.2 (GND), Y1.2 (G), Y1.4 (G)
- new net NRST: C7.1, D1.1 (A1), J1.8 (Pin_8), SW1.1, U1.7 (PG10)
- new net PA0: J3.7 (Pin_7), U1.8 (PA0)
- new net PA1: J3.8 (Pin_8), U1.9 (PA1)
- new net PA10: J3.15 (Pin_15), U1.32 (PA10)
- new net PA11: U1.33 (PA11), U2.6 (I/O1)
- new net PA12: U1.34 (PA12), U2.4 (I/O2)
- new net PA13: J1.3 (Pin_3), U1.37 (PA13)
- new net PA14: J1.4 (Pin_4), U1.38 (PA14)
- new net PA15: J3.16 (Pin_16), U1.39 (PA15)
- new net PA2: J1.6 (Pin_6), U1.10 (PA2)
- new net PA3: J1.5 (Pin_5), U1.11 (PA3)
- new net PA4: J3.9 (Pin_9), U1.12 (PA4)
- new net PA5: J3.10 (Pin_10), U1.13 (PA5)
- new net PA6: J3.11 (Pin_11), U1.14 (PA6)
- new net PA7: J3.12 (Pin_12), U1.15 (PA7)
- new net PA8: J3.13 (Pin_13), U1.30 (PA8)
- new net PA9: J3.14 (Pin_14), U1.31 (PA9)
- new net PB0: J4.5 (Pin_5), U1.16 (PB0)
- new net PB1: J4.6 (Pin_6), U1.17 (PB1)
- new net PB10: J4.15 (Pin_15), U1.22 (PB10)
- new net PB11: J4.16 (Pin_16), U1.25 (PB11)
- new net PB12: J4.17 (Pin_17), U1.26 (PB12)
- new net PB13: J4.18 (Pin_18), U1.27 (PB13)
- new net PB14: J4.19 (Pin_19), U1.28 (PB14)
- new net PB15: J4.20 (Pin_20), U1.29 (PB15)
- new net PB2: J4.7 (Pin_7), R2.1, U1.18 (PB2)
- new net PB3: J4.8 (Pin_8), U1.40 (PB3)
- new net PB4: J4.9 (Pin_9), U1.41 (PB4)
- new net PB5: J4.10 (Pin_10), U1.42 (PB5)
- new net PB6: J4.11 (Pin_11), U1.43 (PB6)
- new net PB7: J4.12 (Pin_12), U1.44 (PB7)
- new net PB9: J4.14 (Pin_14), U1.46 (PB9)
- new net PC13: J3.19 (Pin_19), R3.2, U1.2 (PC13)
- new net PC14: J3.20 (Pin_20), U1.3 (PC14)
- new net PC15: J3.21 (Pin_21), U1.4 (PC15)
- new net PF0: JP1.2 (B), JP3.2 (B), U1.5 (PF0)
- new net PF0_GPIO: J3.17 (Pin_17), JP3.1 (A)
- new net PF1: JP2.2 (B), JP4.2 (B), U1.6 (PF1)
- new net PF1_GPIO: J3.18 (Pin_18), JP4.1 (A)
- new net VBUS: C10.1, C11.1, J2.A4 (VBUS), J2.A9 (VBUS), J2.B4 (VBUS), J2.B9 (VBUS), J4.1 (Pin_1), J4.3 (Pin_3), U2.5 (VBUS)
- new net VDD: C15.1, C3.1, C4.1, C5.1, C6.1, C8.1, C9.1, J1.1 (Pin_1), J3.1 (Pin_1), J3.3 (Pin_3), J3.5 (Pin_5), J4.21 (Pin_21), L1.1, PS1.4 (VOUT), R4.1, SW2.1, SW3.1, U1.1 (VBAT), U1.24 (VDD), U1.36 (VDD), U1.48 (VDD)
- new net VDDA: C1.1, C14.1, C2.1, L1.2, U1.20 (VREF+), U1.21 (VDDA)
- no-connect marks 0 -> 3
Other:
- note added: "ceramic cap (low esr)"

Commit message: changed pin order
Parts:
- removed J3, J4: Conn_02x11_Odd_Even, Connector_PinHeader_2.54mm:PinHeader_2x11_P2.54mm_Vertical, symbol Connector_Generic:Conn_02x11_Odd_Even
- added J3, J4: Conn_01x22, Connector_PinHeader_2.54mm:PinHeader_1x22_P2.54mm_Vertical, symbol Connector_Generic:Conn_01x22
Connections:
- net BOOT0: now also J4.13 (Pin_13)
- net GND: now also J3.22 (Pin_22), J3.4 (Pin_4), J3.5 (Pin_5), J3.6 (Pin_6), J4.22 (Pin_22), J4.3 (Pin_3), J4.4 (Pin_4)
- net PA0: now also J3.12 (Pin_12)
- net PA1: now also J3.13 (Pin_13)
- net PA10: now also J3.20 (Pin_20)
- net PA15: now also J3.21 (Pin_21)
- net PA4: now also J3.14 (Pin_14)
- net PA5: now also J3.15 (Pin_15)
- net PA6: now also J3.16 (Pin_16)
- net PA7: now also J3.17 (Pin_17)
- net PA8: now also J3.18 (Pin_18)
- net PA9: now also J3.19 (Pin_19)
- net PB0: now also J4.5 (Pin_5)
- net PB1: now also J4.6 (Pin_6)
- net PB10: now also J4.15 (Pin_15)
- net PB11: now also J4.16 (Pin_16)
- net PB12: now also J4.17 (Pin_17)
- net PB13: now also J4.18 (Pin_18)
- net PB14: now also J4.19 (Pin_19)
- net PB15: now also J4.20 (Pin_20)
- net PB2: now also J4.7 (Pin_7)
- net PB3: now also J4.8 (Pin_8)
- net PB4: now also J4.9 (Pin_9)
- net PB5: now also J4.10 (Pin_10)
- net PB6: now also J4.11 (Pin_11)
- net PB7: now also J4.12 (Pin_12)
- net PB9: now also J4.14 (Pin_14)
- net PC13: now also J3.9 (Pin_9)
- net PC14: now also J3.10 (Pin_10)
- net PC15: now also J3.11 (Pin_11)
- net PF0_GPIO: now also J3.7 (Pin_7)
- net PF1_GPIO: now also J3.8 (Pin_8)
- net VBUS: now also J4.1 (Pin_1), J4.2 (Pin_2)
- net VDD: now also J3.1 (Pin_1), J3.2 (Pin_2), J3.3 (Pin_3), J4.21 (Pin_21)

Commit message: most routing done
Connections:
- net BOOT0: now also J4.11 (Pin_11); no longer J4.13 (Pin_13)
- net GND: now also J3.1 (Pin_1), J3.17 (Pin_17), J3.18 (Pin_18), J3.19 (Pin_19), J4.19 (Pin_19), J4.2 (Pin_2), J4.20 (Pin_20); no longer J3.22 (Pin_22), J3.4 (Pin_4), J3.5 (Pin_5), J3.6 (Pin_6), J4.22 (Pin_22), J4.3 (Pin_3), J4.4 (Pin_4)
- net PA0: now also J3.7 (Pin_7); no longer J3.12 (Pin_12)
- net PA1: now also J3.8 (Pin_8); no longer J3.13 (Pin_13)
- net PA10: now also J3.15 (Pin_15); no longer J3.20 (Pin_20)
- net PA15: now also J3.16 (Pin_16); no longer J3.21 (Pin_21)
- net PA4: now also J3.9 (Pin_9); no longer J3.14 (Pin_14)
- net PA5: now also J3.10 (Pin_10); no longer J3.15 (Pin_15)
- net PA6: now also J3.11 (Pin_11); no longer J3.16 (Pin_16)
- net PA7: now also J3.12 (Pin_12); no longer J3.17 (Pin_17)
- net PA8: now also J3.13 (Pin_13); no longer J3.18 (Pin_18)
- net PA9: now also J3.14 (Pin_14); no longer J3.19 (Pin_19)
- net PB0: now also J4.3 (Pin_3); no longer J4.5 (Pin_5)
- net PB1: now also J4.4 (Pin_4); no longer J4.6 (Pin_6)
- net PB10: now also J4.13 (Pin_13); no longer J4.15 (Pin_15)
- net PB11: now also J4.14 (Pin_14); no longer J4.16 (Pin_16)
- net PB12: now also J4.15 (Pin_15); no longer J4.17 (Pin_17)
- net PB13: now also J4.16 (Pin_16); no longer J4.18 (Pin_18)
- net PB14: now also J4.17 (Pin_17); no longer J4.19 (Pin_19)
- net PB15: now also J4.18 (Pin_18); no longer J4.20 (Pin_20)
- net PB2: now also J4.5 (Pin_5); no longer J4.7 (Pin_7)
- net PB3: now also J4.6 (Pin_6); no longer J4.8 (Pin_8)
- net PB4: now also J4.7 (Pin_7); no longer J4.9 (Pin_9)
- net PB5: now also J4.8 (Pin_8); no longer J4.10 (Pin_10)
- net PB6: now also J4.9 (Pin_9); no longer J4.11 (Pin_11)
- net PB7: now also J4.10 (Pin_10); no longer J4.12 (Pin_12)
- net PB9: now also J4.12 (Pin_12); no longer J4.14 (Pin_14)
- net PC13: now also J3.4 (Pin_4); no longer J3.9 (Pin_9)
- net PC14: now also J3.5 (Pin_5); no longer J3.10 (Pin_10)
- net PC15: now also J3.6 (Pin_6); no longer J3.11 (Pin_11)
- net PF0_GPIO: now also J3.2 (Pin_2); no longer J3.7 (Pin_7)
- net PF1_GPIO: now also J3.3 (Pin_3); no longer J3.8 (Pin_8)
- net VBUS: now also J4.21 (Pin_21), J4.22 (Pin_22); no longer J4.1 (Pin_1), J4.2 (Pin_2)
- net VDD: now also J3.20 (Pin_20), J3.21 (Pin_21), J3.22 (Pin_22), J4.1 (Pin_1); no longer J3.1 (Pin_1), J3.2 (Pin_2), J3.3 (Pin_3), J4.21 (Pin_21)
